File: schematic/main/main.kicad_sch (KiCad schematic)
At the start: 19 parts, among them J1 Conn_01x01_Pin, J10 Conn_01x01_Pin, J11 Conn_01x01_Pin, J12 Conn_01x01_Pin, J13 Conn_01x01_Pin, J14 Conn_01x01_Pin, J15 Conn_01x01_Pin, J16 Conn_01x01_Pin, J17 Conn_01x01_Pin, J18 Conn_01x01_Pin, J19 Conn_01x01_Pin, J2 Conn_01x01_Pin, J3 Conn_01x01_Pin, J4 Conn_01x01_Pin, J5 Conn_01x01_Pin, J6 Conn_01x01_Pin, J7 Conn_01x01_Pin, J8 Conn_01x01_Pin, J9 Conn_01x01_Pin

Commit message: .
Parts:
- added J22, J6, J7: Conn_01x01_Pin, symbol Connector:Conn_01x01_Pin
- renumbered J8 to J10, J9 to J11, J10 to J12, J11 to J13, J12 to J14, J13 to J15, J14 to J16, J15 to J17, J16 to J18, J17 to J19, J18 to J20, J19 to J21, J6 to J8, J7 to J9
Connections:
- new net +15V: J22.1 (Pin_1)
- new net +5P: J7.1 (Pin_1)
- new net GND: J6.1 (Pin_1)
Other:
- added sheet power (power.kicad_sch)
