File: schematic/main/main.kicad_sch (KiCad schematic)
At the start: 22 parts, among them J1 Conn_01x01_Pin, J10 Conn_01x01_Pin, J11 Conn_01x01_Pin, J12 Conn_01x01_Pin, J13 Conn_01x01_Pin, J14 Conn_01x01_Pin, J15 Conn_01x01_Pin, J16 Conn_01x01_Pin, J17 Conn_01x01_Pin, J18 Conn_01x01_Pin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

Commit message: .
Other:
- added sheet MAX20801 (MAX20801.kicad_sch)
Changed lines of the file:
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@@
+	)
+	(sheet
+		(at 40.64 118.11)
+		(size 45.72 20.32)
+		(exclude_from_sim no)
+		(in_bom yes)
+		(on_board yes)
+		(dnp no)
+		(fields_autoplaced yes)
+		(stroke
+			(width 0.1524)
+			(type solid)
+		)
+		(fill
+			(color 0 0 0 0.0000)
+		)
+		(property "Sheetname" "MAX20801"
+			(at 40.64 117.3984 0)
+			(effects
+				(font
+					(size 1.27 1.27)
+				)
+				(justify left bottom)
+			)
+		)
+		(property "Sheetfile" "MAX20801.kicad_sch"
+			(at 40.64 139.0146 0)
+			(effects
+				(font
+					(size 1.27 1.27)
+				)
+				(justify left top)
+			)
+		)
+		(instances
+			(project "main"
+				(path "/c2b19439-a20b-4150-841d-8b30802ae42a"
+					(page "7")
+				)
+			)
+		)
 	)
 	(sheet
