File: schematic/main/MAX20801.kicad_sch (KiCad schematic)
At the start: 6 parts, among them IC1 MAX20801TPBA+

Commit message: .
Parts:
- added C5, C53, C54, C55, C56, C57, C58, C6: C, symbol common:C
- C1, C3: value C -> 101/2012
Connections:
- net vout: now reaches C2.1, IC1.4 (PV+)
- net vout: now also C4.1, L2.2, C5.1, C53.1, C54.1, C55.1, C56.1, C57.1, C58.1, C6.1
- net +BATT: no longer names the net of C1.1, IC1.1 (VCC)
- net GND renamed gnd
- net gnd: now also C5.2, C53.2, C54.2, C55.2, C56.2, C57.2, C58.2, C6.2
- net out renamed sw
Other:
- moved on the sheet: C2

Commit message: .
Connections:
- net vout: no longer C2.1, C55.1, C56.1, C57.1, C58.1, IC1.4 (PV+)
- new net vin: C2.1, C55.1, C56.1, C57.1, C58.1, IC1.4 (PV+)
