File: schematic/main/analog_buffer.kicad_sch (KiCad schematic)
At the start: 15 parts, among them U3 TLV9362IDGKR

Commit message: .
Parts:
- removed U3: TLV9362IDGKR, Package_SO:VSSOP-8_3x3mm_P0.65mm, symbol common:OPAMP_2CH
- renumbered C7 to C1, C8 to C2, C9 to C3, C10 to C4, C11 to C5, C12 to C6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
Connections:
- net at C1.2, R1.2: now also U1.5 (+); no longer U1.3 (+)
- new net: R3.1, U1.6 (-), U1.7
Other:
- moved on the sheet: C2

Commit message: .
Parts:
- renumbered D1 to D4, D2 to D5, R1 to R4, R2 to R5, R3 to R6, R4 to R7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
