File: schematic/main/high_voltage.kicad_sch (KiCad schematic)
At the start: 47 parts, among them U2 TLV9362IDGKR, U3 AMC3330, U4 AMC3330

Commit message: .
Parts:
- renumbered U2 to U1, U3 to U2, U2 to U3
Connections:
- net A-5V: now also U1.4 (V-)
- net GNDA: no longer U1.4 (V-)
Other:
- moved on the sheet: U1C
Changed lines of the file:
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@@
 		(dnp no)
 		(fields_autoplaced yes)
-		(property "Reference" "#PWR027"
+		(property "Reference" "#PWR026"
 			(at 208.28 38.1 0)
 			(effects
@@
 			(project "main"
 				(path "/c2b19439-a20b-4150-841d-8b30802ae42a/e2ee3a16-f48b-4c51-9225-da559e7c02f4"
-					(reference "#PWR027")
+					(reference "#PWR026")
 					(unit 1)
 				)
@@
 	)
 	(symbol
-		(lib_id "power:GNDA")
-		(at 247.65 54.61 0)
-		(unit 1)
-		(exclude_from_sim no)
-		(in_bom yes)
-		(on_board yes)
-		(dnp no)
-		(fields_autoplaced yes)
-		(property "Reference" "#PWR030"
-			(at 247.65 60.96 0)
-			(effects
-				(font
-					(size 1.27 1.27)
-				)
-				(hide yes)
-			)
-		)
-		(property "Value" "GNDA"
-			(at 247.65 59.69 0)
-			(effects
-				(font
-					(size 1.27 1.27)
-				)
-			)
-		)
-		(property "Footprint" ""
-			(at 247.65 54.61 0)
-			(effects
-				(font
-					(size 1.27 1.27)
-				)
-				(hide yes)
-			)
-		)
-		(property "Datasheet" ""
-			(at 247.65 54.61 0)
-			(effects
-				(font
-					(size 1.27 1.27)
-				)
-				(hide yes)
-			)
-		)
-		(property "Description" "Power symbol creates a global label with name \"GNDA\" , analog ground"
-			(at 247.65 54.61 0)
-			(effects
-				(font
-					(size 1.27 1.27)
-				)
-				(hide yes)
-			)
-		)
-		(pin "1"
-		)
-		(instances
-			(project "main"
-				(path "/c2b19439-a20b-4150-841d-8b30802ae42a/e2ee3a16-f48b-4c51-9225-da559e7c02f4"
-					(reference "#PWR030")
-					(unit 1)
-				)
-			)
-		)
-	)
-	(symbol
 		(lib_id "common:C")
 		(at 76.2 109.22 0)
@@
 		(dnp no)
 		(fields_autoplaced yes)
-		(property "Reference" "U3"
+		(property "Reference" "U2"
 			(at 140.5733 33.02 0)
 			(effects
@@
 			(project "main"
 				(path "/c2b19439-a20b-4150-841d-8b30802ae42a/e2ee3a16-f48b-4c51-9225-da559e7c02f4"
-					(reference "U3")
+					(reference "U2")
 					(unit 1)
 				)
@@
 		(dnp no)
 		(fields_autoplaced yes)
-		(property "Reference" "#PWR024"
+		(property "Reference" "#PWR023"
 			(at 180.34 46.99 0)
 			(effects
@@
 			(project "main"
 				(path "/c2b19439-a20b-4150-841d-8b30802ae42a/e2ee3a16-f48b-4c51-9225-da559e7c02f4"
-					(reference "#PWR024")
+					(reference "#PWR023")
 					(unit 1)
 				)
@@
 		(dnp no)
 		(fields_autoplaced yes)
-		(property "Reference" "#FLG06"
+		(property "Reference" "#FLG08"
 			(at 109.22 75.565 0)
 			(effects
@@
 			(project ""
 				(path "/c2b19439-a20b-4150-841d-8b30802ae42a/e2ee3a16-f48b-4c51-9225-da559e7c02f4"
-					(reference "#FLG06")
+					(reference "#FLG08")
 					(unit 1)
 				)
@@
 		(dnp no)
 		(fields_autoplaced yes)
-		(property "Reference" "#PWR028"
+		(property "Reference" "#PWR027"
 			(at 218.44 38.1 0)
 			(effects
@@
 			(project "main"
 				(path "/c2b19439-a20b-4150-841d-8b30802ae42a/e2ee3a16-f48b-4c51-9225-da559e7c02f4"
-					(reference "#PWR028")
+					(reference "#PWR027")
+					(unit 1)
+				)
+			)
+		)
+	)
+	(symbol
+		(lib_id "power:-5V")
+		(at 266.7 92.71 180)
+		(unit 1)
+		(exclude_from_sim no)
+		(in_bom yes)
+		(on_board yes)
+		(dnp no)
+		(fields_autoplaced yes)
+		(property "Reference" "#PWR032"
+			(at 266.7 88.9 0)
+			(effects
+				(font
+					(size 1.27 1.27)
+				)
+				(hide yes)
+			)
+		)
+		(property "Value" "A-5V"
+			(at 266.7 97.79 0)
+			(effects
+				(font
+					(size 1.27 1.27)
+				)
+			)
+		)
+		(property "Footprint" ""
+			(at 266.7 92.71 0)
+			(effects
+				(font
+					(size 1.27 1.27)
+				)
+				(hide yes)
+			)
+		)
+		(property "Datasheet" ""
+			(at 266.7 92.71 0)
+			(effects
+				(font
+					(size 1.27 1.27)
+				)
+				(hide yes)
+			)
+		)
+		(property "Description" "Power symbol creates a global label with name \"-5V\""
+			(at 266.7 92.71 0)
+			(effects
+				(font
+					(size 1.27 1.27)
+				)
+				(hide yes)
+			)
+		)
+		(pin "1"
+		)
+		(instances
+			(project "main"
+				(path "/c2b19439-a20b-4150-841d-8b30802ae42a/e2ee3a16-f48b-4c51-9225-da559e7c02f4"
+					(reference "#PWR032")
 					(unit 1)
 				)
@@
 		(dnp no)
 		(fields_autoplaced yes)
-		(property "Reference" "#PWR026"
+		(property "Reference" "#PWR025"
 			(at 76.2 50.8 0)
 			(effects
@@
 			(project "main"
 				(path "/c2b19439-a20b-4150-841d-8b30802ae42a/e2ee3a16-f48b-4c51-9225-da559e7c02f4"
-					(reference "#PWR026")
+					(reference "#PWR025")
 					(unit 1)
 				)
@@
 	(symbol
 		(lib_id "power:+5V")
-		(at 247.65 39.37 0)
+		(at 266.7 77.47 0)
 		(unit 1)
 		(exclude_from_sim no)
@@
 		(dnp no)
 		(fields_autoplaced yes)
-		(property "Reference" "#PWR023"
-			(at 247.65 43.18 0)
+		(property "Reference" "#PWR030"
+			(at 266.7 81.28 0)
 			(effects
 				(font
@@
 		)
 		(property "Value" "A+5V"
-			(at 247.65 34.29 0)
+			(at 266.7 72.39 0)
 			(effects
 				(font
@@
 		)
 		(property "Footprint" ""
-			(at 247.65 39.37 0)
+			(at 266.7 77.47 0)
 			(effects
 				(font
@@
 		)
 		(property "Datasheet" ""
-			(at 247.65 39.37 0)
+			(at 266.7 77.47 0)
 			(effects
 				(font
@@
 		)
 		(property "Description" "Power symbol creates a global label with name \"+5V\""
-			(at 247.65 39.37 0)
+			(at 266.7 77.47 0)
 			(effects
 				(font
@@
 			(project "main"
 				(path "/c2b19439-a20b-4150-841d-8b30802ae42a/e2ee3a16-f48b-4c51-9225-da559e7c02f4"
-					(reference "#PWR023")
+					(reference "#PWR030")
 					(unit 1)
 				)
@@
 	(symbol
 		(lib_id "common:OPAMP_2CH")
-		(at 250.19 46.99 0)
+		(at 269.24 85.09 0)
 		(unit 3)
 		(exclude_from_sim no)
@@
 		(dnp no)
 		(fields_autoplaced yes)
-		(property "Reference" "U2"
-			(at 248.92 45.7199 0)
+		(property "Reference" "U1"
+			(at 267.97 83.8199 0)
 			(effects
 				(font
@@
 		)
 		(property "Value" "TLV9362IDGKR"
-			(at 248.92 48.2599 0)
+			(at 267.97 86.3599 0)
 			(effects
 				(font
@@
 		)
 		(property "Footprint" "Package_SO:VSSOP-8_3x3mm_P0.65mm"
-			(at 250.19 46.99 0)
+			(at 269.24 85.09 0)
 			(effects
 				(font
@@
 		)
 		(property "Datasheet" "http://www.ti.com/lit/ds/symlink/lm358.pdf"
-			(at 250.19 46.99 0)
+			(at 269.24 85.09 0)
 			(effects
 				(font
@@
 		)
 		(property "Description" "Dual Operational Amplifiers, DIP-8/SOIC-8/TSSOP-8/VSSOP-8"
-			(at 250.19 46.99 0)
+			(at 269.24 85.09 0)
 			(effects
 				(font
@@
 		)
 		(property "Part Number" ""
-			(at 250.19 46.99 0)
+			(at 269.24 85.09 0)
 			(effects
 				(font
@@
 		)
 		(property "Manfacturer" ""
-			(at 250.19 46.99 0)
+			(at 269.24 85.09 0)
 			(effects
 				(font
@@
 		)
 		(property "Cost" ""
-			(at 250.19 46.99 0)
+			(at 269.24 85.09 0)
 			(effects
 				(font
@@
 			(project ""
 				(path "/c2b19439-a20b-4150-841d-8b30802ae42a/e2ee3a16-f48b-4c51-9225-da559e7c02f4"
-					(reference "U2")
+					(reference "U1")
 					(unit 3)
 				)
@@
 		(dnp no)
 		(fields_autoplaced yes)
-		(property "Reference" "#PWR029"
+		(property "Reference" "#PWR028"
 			(at 158.75 52.07 0)
 			(effects
@@
 			(project "main"
 				(path "/c2b19439-a20b-4150-841d-8b30802ae42a/e2ee3a16-f48b-4c51-9225-da559e7c02f4"
-					(reference "#PWR029")
+					(reference "#PWR028")
 					(unit 1)
 				)
@@
 		(dnp no)
 		(fields_autoplaced yes)
-		(property "Reference" "#PWR032"
+		(property "Reference" "#PWR031"
 			(at 243.84 86.36 0)
 			(effects
@@
 			(project "main"
 				(path "/c2b19439-a20b-4150-841d-8b30802ae42a/e2ee3a16-f48b-4c51-9225-da559e7c02f4"
-					(reference "#PWR032")
+					(reference "#PWR031")
 					(unit 1)
 				)
@@
 		(dnp no)
 		(fields_autoplaced yes)
-		(property "Reference" "#FLG07"
+		(property "Reference" "#FLG09"
 			(at 105.41 145.415 0)
 			(effects
@@
 			(project "main"
 				(path "/c2b19439-a20b-4150-841d-8b30802ae42a/e2ee3a16-f48b-4c51-9225-da559e7c02f4"
-					(reference "#FLG07")
+					(reference "#FLG09")
 					(unit 1)
 				)
@@
 		(dnp no)
 		(fields_autoplaced yes)
-		(property "Reference" "U2"
+		(property "Reference" "U3"
 			(at 214.63 128.27 0)
 			(effects
@@
 			(project ""
 				(path "/c2b19439-a20b-4150-841d-8b30802ae42a/e2ee3a16-f48b-4c51-9225-da559e7c02f4"
-					(reference "U2")
+					(reference "U3")
 					(unit 2)
 				)
@@
 		(dnp no)
 		(fields_autoplaced yes)
-		(property "Reference" "U2"
+		(property "Reference" "U3"
 			(at 215.9 58.42 0)
 			(effects
@@
 			(project ""
 				(path "/c2b19439-a20b-4150-841d-8b30802ae42a/e2ee3a16-f48b-4c51-9225-da559e7c02f4"
-					(reference "U2")
+					(reference "U3")
 					(unit 1)
 				)
@@
 		(dnp no)
 		(fields_autoplaced yes)
-		(property "Reference" "#PWR031"
+		(property "Reference" "#PWR029"
 			(at 138.43 80.01 0)
 			(effects
@@
 			(project "main"
 				(path "/c2b19439-a20b-4150-841d-8b30802ae42a/e2ee3a16-f48b-4c51-9225-da559e7c02f4"
-					(reference "#PWR031")
+					(reference "#PWR029")
 					(unit 1)
 				)
@@
 		(dnp no)
 		(fields_autoplaced yes)
-		(property "Reference" "#PWR025"
+		(property "Reference" "#PWR024"
 			(at 64.77 50.8 0)
 			(effects
@@
 			(project "main"
 				(path "/c2b19439-a20b-4150-841d-8b30802ae42a/e2ee3a16-f48b-4c51-9225-da559e7c02f4"
-					(reference "#PWR025")
+					(reference "#PWR024")
 					(unit 1)
 				)

Commit message: .
Parts:
- C20: value 102 -> 105
Connections:
- net hgnd0: now reaches C11.1, C12.1, C14.1, C15.1, C8.1, U2.2 (DCDC_HGND)
- net hgnd0: now also C16.1, R12.2, U2.7 (INN), U2.8 (HGND)
- net hgnd1: now reaches C30.1, R21.2, U4.7 (INN), U4.8 (HGND)
- net hgnd1: now also C22.1, C25.1, C26.1, C28.1, C29.1, U4.2 (DCDC_HGND)
Changed lines of the file:
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@@
 	)
 	(junction
-		(at 109.22 77.47)
-		(diameter 0)
-		(color 0 0 0 0)
-	)
-	(junction
 		(at 59.69 77.47)
 		(diameter 0)
@@
 	)
 	(junction
-		(at 105.41 147.32)
+		(at 59.69 69.85)
 		(diameter 0)
 		(color 0 0 0 0)
 	)
 	(junction
-		(at 59.69 69.85)
+		(at 207.01 132.08)
 		(diameter 0)
 		(color 0 0 0 0)
 	)
 	(junction
-		(at 207.01 132.08)
+		(at 96.52 57.15)
 		(diameter 0)
 		(color 0 0 0 0)
 	)
 	(junction
-		(at 96.52 57.15)
+		(at 96.52 77.47)
 		(diameter 0)
 		(color 0 0 0 0)
@@
 	)
 	(junction
+		(at 95.25 134.62)
+		(diameter 0)
+		(color 0 0 0 0)
+	)
+	(junction
 		(at 226.06 83.82)
 		(diameter 0)
@@
 	)
 	(junction
+		(at 96.52 64.77)
+		(diameter 0)
+		(color 0 0 0 0)
+	)
+	(junction
 		(at 58.42 147.32)
 		(diameter 0)
@@
 		(color 0 0 0 0)
 	)
+	(junction
+		(at 95.25 147.32)
+		(diameter 0)
+		(color 0 0 0 0)
+	)
 	(wire
 		(pts
@@
 	(wire
 		(pts
-			(xy 105.41 147.32) (xy 114.3 147.32)
+			(xy 95.25 147.32) (xy 114.3 147.32)
 		)
 		(stroke
@@
 	(wire
 		(pts
+			(xy 96.52 64.77) (xy 96.52 77.47)
+		)
+		(stroke
+			(width 0)
+			(type default)
+		)
+	)
+	(wire
+		(pts
 			(xy 207.01 162.56) (xy 207.01 152.4)
 		)
@@
 	(wire
 		(pts
-			(xy 91.44 147.32) (xy 105.41 147.32)
+			(xy 91.44 147.32) (xy 95.25 147.32)
 		)
 		(stroke
@@
 	(wire
 		(pts
+			(xy 95.25 134.62) (xy 95.25 147.32)
+		)
+		(stroke
+			(width 0)
+			(type default)
+		)
+	)
+	(wire
+		(pts
 			(xy 59.69 69.85) (xy 80.01 69.85)
 		)
@@
 	(wire
 		(pts
-			(xy 109.22 77.47) (xy 115.57 77.47)
+			(xy 96.52 77.47) (xy 115.57 77.47)
 		)
 		(stroke
@@
 	(wire
 		(pts
-			(xy 92.71 77.47) (xy 109.22 77.47)
+			(xy 92.71 77.47) (xy 96.52 77.47)
 		)
 		(stroke
@@
 		)
 	)
+	(label "hgnd0"
+		(at 102.87 77.47 0)
+		(effects
+			(font
+				(size 1.27 1.27)
+			)
+			(justify left bottom)
+		)
+	)
+	(label "hgnd1"
+		(at 101.6 147.32 0)
+		(effects
+			(font
+				(size 1.27 1.27)
+			)
+			(justify left bottom)
+		)
+	)
 	(hierarchical_label "vac_n0"
 		(shape bidirectional)
@@
 			)
 		)
-		(property "Value" "102"
+		(property "Value" "105"
 			(at 243.078 100.584 0)
 			(effects
@@
 	)
 	(symbol
-		(lib_id "power:PWR_FLAG")
-		(at 109.22 77.47 0)
-		(unit 1)
-		(exclude_from_sim no)
-		(in_bom yes)
-		(on_board yes)
-		(dnp no)
-		(fields_autoplaced yes)
-		(property "Reference" "#FLG08"
-			(at 109.22 75.565 0)
-			(effects
-				(font
-					(size 1.27 1.27)
-				)
-				(hide yes)
-			)
-		)
-		(property "Value" "PWR_FLAG"
-			(at 109.22 72.39 0)
-			(effects
-				(font
-					(size 1.27 1.27)
-				)
-			)
-		)
-		(property "Footprint" ""
-			(at 109.22 77.47 0)
-			(effects
-				(font
-					(size 1.27 1.27)
-				)
-				(hide yes)
-			)
-		)
-		(property "Datasheet" "~"
-			(at 109.22 77.47 0)
-			(effects
-				(font
-					(size 1.27 1.27)
-				)
-				(hide yes)
-			)
-		)
-		(property "Description" "Special symbol for telling ERC where power comes from"
-			(at 109.22 77.47 0)
-			(effects
-				(font
-					(size 1.27 1.27)
-				)
-				(hide yes)
-			)
-		)
-		(pin "1"
-		)
-		(instances
-			(project ""
-				(path "/c2b19439-a20b-4150-841d-8b30802ae42a/e2ee3a16-f48b-4c51-9225-da559e7c02f4"
-					(reference "#FLG08")
-					(unit 1)
-				)
-			)
-		)
-	)
-	(symbol
 		(lib_id "common:R_US")
 		(at 83.82 77.47 90)
@@
 					(unit 1)
 				)
-			)
-		)
-	)
-	(symbol
-		(lib_id "power:PWR_FLAG")
-		(at 105.41 147.32 0)
-		(unit 1)
-		(exclude_from_sim no)
-		(in_bom yes)
-		(on_board yes)
-		(dnp no)
-		(fields_autoplaced yes)
-		(property "Reference" "#FLG09"
-			(at 105.41 145.415 0)
-			(effects
-				(font
-					(size 1.27 1.27)
-				)
-				(hide yes)
-			)
-		)
-		(property "Value" "PWR_FLAG"
-			(at 105.41 142.24 0)
-			(effects
-				(font
-					(size 1.27 1.27)
-				)
-			)
-		)
-		(property "Footprint" ""
-			(at 105.41 147.32 0)
-			(effects
-				(font
-					(size 1.27 1.27)
-				)
-				(hide yes)
-			)
-		)
-		(property "Datasheet" "~"
-			(at 105.41 147.32 0)
-			(effects
-				(font
-					(size 1.27 1.27)
-				)
-				(hide yes)
-			)
-		)
-		(property "Description" "Special symbol for telling ERC where power comes from"
-			(at 105.41 147.32 0)
-			(effects
-				(font
-					(size 1.27 1.27)
-				)
-				(hide yes)
-			)
-		)
-		(pin "1"
-		)
-		(instances
-			(project "main"
-				(path "/c2b19439-a20b-4150-841d-8b30802ae42a/e2ee3a16-f48b-4c51-9225-da559e7c02f4"
-					(reference "#FLG09")
-					(unit 1)
-				)
